File: CAD/uplc-digital/uplc-digital.kicad_pcb (KiCad board)
At the start: 4 copper layers, 31.4 x 21 mm, 54 parts, among them J1 Conn_01x06_Pin, J2 SM12B-GHS-TB(LF)(SN), U1 AP63201WU, U2 TBD62003AFWG, U3 ESP32-C3-WROOM-02, Y1 32.768khz 3215 12.5pf

Commit message: WIP rev 1.1
Parts:
- removed R10, R11, R12, R3, R7, R8, R9: 10K, Resistor_SMD:R_0402_1005Metric
- added JP1: J3O, Jumper:SolderJumper-3_P1.3mm_Open_Pad1.0x1.5mm_NumberLabels, F.Cu at (108.2, 79.5)
- added JP10: J3O, Jumper:SolderJumper-3_P1.3mm_Open_Pad1.0x1.5mm_NumberLabels, F.Cu at (121.2, 85.8)
- added JP11: J3O, Jumper:SolderJumper-3_P1.3mm_Open_Pad1.0x1.5mm_NumberLabels, F.Cu at (121.2, 87.9)
- added JP12: J3O, Jumper:SolderJumper-3_P1.3mm_Open_Pad1.0x1.5mm_NumberLabels, F.Cu at (121.2, 90.0)
- added JP2: J3O, Jumper:SolderJumper-3_P1.3mm_Open_Pad1.0x1.5mm_NumberLabels, F.Cu at (108.2, 81.6)
- added JP3: J3O, Jumper:SolderJumper-3_P1.3mm_Open_Pad1.0x1.5mm_NumberLabels, F.Cu at (108.2, 83.7)
- added JP4: J3O, Jumper:SolderJumper-3_P1.3mm_Open_Pad1.0x1.5mm_NumberLabels, F.Cu at (108.2, 85.8)
- added JP5: J3O, Jumper:SolderJumper-3_P1.3mm_Open_Pad1.0x1.5mm_NumberLabels, F.Cu at (108.2, 87.9)
- added JP6: J3O, Jumper:SolderJumper-3_P1.3mm_Open_Pad1.0x1.5mm_NumberLabels, F.Cu at (108.2, 90.0)
- added JP7: J3O, Jumper:SolderJumper-3_P1.3mm_Open_Pad1.0x1.5mm_NumberLabels, F.Cu at (121.2, 79.5)
- added JP8: J3O, Jumper:SolderJumper-3_P1.3mm_Open_Pad1.0x1.5mm_NumberLabels, F.Cu at (121.2, 81.6)
- added JP9: J3O, Jumper:SolderJumper-3_P1.3mm_Open_Pad1.0x1.5mm_NumberLabels, F.Cu at (121.2, 83.7)
- moved C12 20.2 mm to (138.9, 69.5)
- moved C9 20.2 mm to (144.3, 64.7)
- moved D4 20.2 mm to (141.2, 64.3)
- moved C2 20.2 mm to (143.3, 68.4)
- moved C5 20.2 mm to (138.4, 66.9)
- moved L1 20.2 mm to (141.7, 70.8)
- moved R14 20.2 mm to (143.3, 64.7)
- moved R15 20.2 mm to (143.3, 66.6)
- moved U1 20.2 mm to (141.1, 67.2)
- moved C8 20.2 mm to (137.9, 69.5)
- moved R5 15.8 mm to (111.5, 73.8)
- moved C1 4.41 mm to (107.0, 76.3), turned to -90 degrees
- moved C4 4.38 mm to (112.0, 76.3), turned to 90 degrees
- moved R6 3.16 mm to (122.6, 91.8), turned to 0 degrees
- moved U2 2.84 mm to (114.8, 85.9)
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Connections:
- U2 pad 1: LI1 -> Net-(JP1-C)
- U2 pad 10: HO5 -> unconnected-(U2-O7-Pad10)
- U2 pad 11: LO7 -> Net-(JP12-C)
- U2 pad 12: LO6 -> Net-(JP11-C)
- U2 pad 13: HO4 -> Net-(JP10-C)
- U2 pad 14: HO3 -> Net-(JP9-C)
- U2 pad 15: HO2 -> Net-(JP8-C)
- U2 pad 16: HO1 -> Net-(JP7-C)
- U2 pad 2: LI2 -> Net-(JP2-C)
- U2 pad 3: LI3 -> Net-(JP3-C)
- U2 pad 4: LI4 -> Net-(JP4-C)
- U2 pad 5: HI1 -> Net-(JP5-C)
- U2 pad 6: HI2 -> Net-(JP6-C)
- U2 pad 7: LI5 -> unconnected-(U2-I7-Pad7)
Routing:
- net +3.3V: track 88.5 -> 0.00 mm, vias 13 -> 10
- net GND: track 26.7 -> 0.00 mm, vias 49 -> 13
- net HI2: track 21.7 -> 0.00 mm, vias 3 -> 0
- net HI1: track 21.4 -> 0.00 mm, vias 3 -> 0
- net RST: track 19.2 -> 0.00 mm, vias 2 -> 0
- net Net-(U3-GPIO1/ADC1_CH1/XTAL_32K_N): track 18.2 -> 0.00 mm, vias 1 -> 0
- net HO1: track 15.5 -> 0.00 mm, vias 2 -> 0
- net HO2: track 15.2 -> 0.00 mm, vias 2 -> 0
- net Net-(U3-GPIO0/ADC1_CH0/XTAL_32K_P): track 13.9 -> 0.00 mm, vias 1 -> 0
- net ONEWIRE: track 12.8 -> 0.00 mm, vias 1 -> 0
- net LI4: track 11.7 -> 0.00 mm, vias 1 -> 0
- net LI3: track 11.0 -> 0.00 mm, vias 1 -> 0
- net LO6: track 10.2 -> 0.00 mm, vias 1 -> 0
- net LI2: track 9.85 -> 0.00 mm, vias 1 -> 0
- net BOOT: track 9.64 -> 0.00 mm, vias 1 -> 0
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
Commit message: Rev 1.1 Schem PCB done
Parts:
- removed kibuzzard-65D3619D: G***, esprelay:kibuzzard-65D3619D
- removed kibuzzard-65D361A7: G***, esprelay:kibuzzard-65D361A7
- removed kibuzzard-65D361B0: G***, esprelay:kibuzzard-65D361B0
- removed kibuzzard-65D361D3: G***, esprelay:kibuzzard-65D361D3
- removed kibuzzard-65D736F5: G***, kibuzzard-65D736F5
- removed kibuzzard-65D74DB4: G***, kibuzzard-65D74DB4
- removed kibuzzard-65D74DBE: G***, kibuzzard-65D74DBE
- removed kibuzzard-65D74DD6: G***, kibuzzard-65D74DD6
- added D3: 1N5819WS, Diode_SMD:D_SOD-323, F.Cu at (111.5, 74.3)
- added R3: 10K, Resistor_SMD:R_0402_1005Metric, F.Cu at (111.0, 76.8)
- added R7: 309k, Resistor_SMD:R_0402_1005Metric, F.Cu at (112.0, 76.8)
- added kibuzzard-65D8B0E2: G***, kibuzzard-65D8B0E2, B.Cu at (128.4, 77.1)
- added kibuzzard-65D8B0ED: G***, kibuzzard-65D8B0ED, B.Cu at (128.4, 78.7)
- added kibuzzard-65D8B0F8: G***, kibuzzard-65D8B0F8, B.Cu at (128.4, 80.2)
- added kibuzzard-65D8B104: G***, kibuzzard-65D8B104, B.Cu at (128.4, 81.8)
- added kibuzzard-65D8B10C: G***, kibuzzard-65D8B10C, B.Cu at (128.4, 83.3)
- added kibuzzard-65D8B121: G***, kibuzzard-65D8B121, B.Cu at (128.4, 84.9)
- added kibuzzard-65D8B28C: G***, kibuzzard-65D8B28C, F.Cu at (109.4, 79.1)
- added kibuzzard-65D8B297: G***, kibuzzard-65D8B297, F.Cu at (119.5, 79.2)
- added kibuzzard-65D8B2B0: G***, kibuzzard-65D8B2B0, F.Cu at (104.5, 82.6)
- added kibuzzard-65D8B343: G***, kibuzzard-65D8B343, B.Cu at (128.4, 86.4)
- JP1, JP10, JP11, JP12, JP2, JP3, JP4, JP5, JP6, JP7, JP8, JP9: value J3O -> 0R; footprint Jumper:SolderJumper-3_P1.3mm_Open_Pad1.0x1.5mm_NumberLabels -> Jumper:SolderJumper-3_P1.3mm_BridgedSMD12_0402
- moved C2 25.5 mm to (119.6, 78.1), turned to 0 degrees
- moved C9 25.4 mm to (123.3, 79.1), turned to 180 degrees
- moved L1 25.1 mm to (117.2, 76.5), turned to 90 degrees
- moved R15 24.6 mm to (121.5, 78.1), turned to 0 degrees
- moved R14 24.0 mm to (123.3, 78.1), turned to 0 degrees
- moved U1 22.0 mm to (120.8, 75.9), turned to 180 degrees
- moved D4 21.0 mm to (123.7, 76.0), turned to -90 degrees
- moved C12 20.7 mm to (118.6, 73.7), turned to 0 degrees
- moved C8 19.7 mm to (118.6, 72.7), turned to 0 degrees
- moved C5 18.3 mm to (121.2, 73.2), turned to 180 degrees
- moved R5 17.4 mm to (111.5, 91.2), turned to -90 degrees
- moved Y1 14.7 mm to (108.9, 91.2)
- moved JP6 14.0 mm to (120.3, 82.9)
- moved C4 13.4 mm to (109.2, 89.4), turned to 0 degrees
- moved C1 13.1 mm to (107.3, 89.4), turned to 0 degrees
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Connections:
- net Net-(JP1-C) renamed /I1
- J2 pad 10: HO1 -> H1
- J2 pad 4: HO5 -> GND
- J2 pad 5: HO4 -> H6
- J2 pad 6: HO3 -> H5
- J2 pad 7: HI2 -> H4
- J2 pad 8: HI1 -> H3
- J2 pad 9: HO2 -> H2
- JP1 pad 1: unconnected-(JP1-A-Pad1) -> H1
- JP1 pad 3: unconnected-(JP1-B-Pad3) -> L1
- JP10 pad 1: unconnected-(JP10-A-Pad1) -> H5
- JP10 pad 2: Net-(JP10-C) -> /O5
- JP10 pad 3: unconnected-(JP10-B-Pad3) -> L5
- JP11 pad 1: unconnected-(JP11-A-Pad1) -> L6
- JP11 pad 2: Net-(JP11-C) -> /I6
- JP11 pad 3: unconnected-(JP11-B-Pad3) -> H6
- JP12 pad 1: unconnected-(JP12-A-Pad1) -> H6
- JP12 pad 2: Net-(JP12-C) -> /O6
- JP12 pad 3: unconnected-(JP12-B-Pad3) -> L6
- JP2 pad 1: unconnected-(JP2-A-Pad1) -> L1
- JP2 pad 2: Net-(JP2-C) -> /O1
- JP2 pad 3: unconnected-(JP2-B-Pad3) -> H1
- JP3 pad 1: unconnected-(JP3-A-Pad1) -> H2
- JP3 pad 2: Net-(JP3-C) -> /I2
- JP3 pad 3: unconnected-(JP3-B-Pad3) -> L2
- JP4 pad 1: unconnected-(JP4-A-Pad1) -> L2
- JP4 pad 2: Net-(JP4-C) -> /O2
- JP4 pad 3: unconnected-(JP4-B-Pad3) -> H2
- JP5 pad 1: unconnected-(JP5-A-Pad1) -> H3
- JP5 pad 2: Net-(JP5-C) -> /I3
- JP5 pad 3: unconnected-(JP5-B-Pad3) -> L3
- JP6 pad 1: unconnected-(JP6-A-Pad1) -> L3
- JP6 pad 2: Net-(JP6-C) -> /O3
- JP6 pad 3: unconnected-(JP6-B-Pad3) -> H3
- JP7 pad 1: unconnected-(JP7-A-Pad1) -> L4
- JP7 pad 2: Net-(JP7-C) -> /I4
- JP7 pad 3: unconnected-(JP7-B-Pad3) -> H4
- JP8 pad 1: unconnected-(JP8-A-Pad1) -> H4
- JP8 pad 2: Net-(JP8-C) -> /O4
- JP8 pad 3: unconnected-(JP8-B-Pad3) -> L4
- JP9 pad 1: unconnected-(JP9-A-Pad1) -> L5
- JP9 pad 2: Net-(JP9-C) -> /I5
- JP9 pad 3: unconnected-(JP9-B-Pad3) -> H5
- U2 pad 10: unconnected-(U2-O7-Pad10) -> /O6
- U2 pad 11: Net-(JP12-C) -> /O6
- U2 pad 12: Net-(JP11-C) -> /O5
- U2 pad 13: Net-(JP10-C) -> /O4
- U2 pad 14: Net-(JP9-C) -> /O3
- U2 pad 15: Net-(JP8-C) -> /O2
- U2 pad 16: Net-(JP7-C) -> /O1
- U2 pad 2: Net-(JP2-C) -> /I2
- U2 pad 3: Net-(JP3-C) -> /I3
- U2 pad 4: Net-(JP4-C) -> /I4
- U2 pad 5: Net-(JP5-C) -> /I5
- U2 pad 6: Net-(JP6-C) -> /I6
- U2 pad 7: unconnected-(U2-I7-Pad7) -> /I6
- U3 pad 10: LO7 -> L6
- U3 pad 14: LO6 -> L5
- U3 pad 15: LI5 -> L4
- U3 pad 3: LI4 -> ADC
- U3 pad 4: LI3 -> L1
- U3 pad 5: LI2 -> L2
- U3 pad 6: LI1 -> L3
Routing:
- net GND: track 0.00 -> 81.8 mm, vias 13 -> 62
- net +3.3V: track 0.00 -> 78.9 mm, vias 10 -> 9
- net L6: track 0.00 -> 28.8 mm, vias 0 -> 1
- net H5: track 0.00 -> 23.9 mm, vias 0 -> 2
- net L3: track 0.00 -> 23.7 mm, vias 0 -> 1
- net H4: track 0.00 -> 23.1 mm, vias 0 -> 2
- net H6: track 0.00 -> 23.1 mm, vias 0 -> 2
- net H3: track 0.00 -> 22.8 mm, vias 0 -> 2
- net H2: track 0.00 -> 22.8 mm, vias 0 -> 2
- net H1: track 0.00 -> 22.5 mm, vias 0 -> 2
- net L2: track 0.00 -> 21.7 mm, vias 0 -> 1
- net L4: track 0.00 -> 20.9 mm, vias 0 -> 1
- net L1: track 0.00 -> 20.2 mm, vias 0 -> 1
- net RST: track 0.00 -> 20.2 mm, vias 0 -> 2
- net BOOT: track 0.00 -> 18.1 mm, vias 0 -> 1
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- added copper zone on In1.Cu, net +3.3V
- added copper zone on In2.Cu, net H6
- removed copper zone on In2.Cu, net +3.3V
- removed copper zone on In2.Cu, net HO1
- removed copper zone on In2.Cu, net HO2

Commit message: Rev 1.1 Push for production
Routing:
- net GND: track 81.8 -> 83.7 mm
- net L5: track 16.9 -> 16.0 mm
- net Net-(U3-GPIO1/ADC1_CH1/XTAL_32K_N): track 5.86 -> 5.10 mm
- net +3.3V: track 78.9 -> 78.1 mm
- net /O6: track 8.56 -> 9.08 mm
- removed copper zone on In2.Cu, net H6
Other:
- board text added: "1"
- board text added: "2"
- board text added: "3"
- board text added: "4"
- board text added: "6"

Commit message: Rev 1.2
Parts:
- removed kibuzzard-65D8B2B0: G***, kibuzzard-65D8B2B0
- added kibuzzard-65DCA831: G***, kibuzzard-65DCA831, F.Cu at (104.5, 82.6)
Connections:
- U3 pad 13: ONEWIRE -> L4
- U3 pad 15: L4 -> ONEWIRE
Routing:
- net ONEWIRE: track 14.3 -> 16.7 mm
- net L4: track 20.8 -> 19.5 mm
- net GND: track 83.7 -> 82.9 mm

Commit message: Panelization changes
Routing:
- net GND: track 82.9 -> 84.9 mm
Other:
- board size 31.4 x 21 mm -> 31.4 x 22 mm

Commit message: Feat: V1.1
Parts:
- L1: value 6.8uH -> 4.7uH
